File: hardware/kicad/posture_tracker_v2/posture_tracker_v2/posture_tracker_v2.kicad_sch (KiCad schematic)
At the start: 52 parts, among them J1 HRO TYPE-C-31-M-12, J2 JST-PH-2, M1 Molex_PicoBlade_53047-0210, SW1 BTN_CAL, SW2 BTN_SNOOZE, SW3 RESET, U1 ESP32-S3-MINI-1, U2 MPU-6050, U3 DRV2605LDGS, U4 MAX98357A, U5 MCP73831T-2ACI/OT, U6 AP2112K-3.3TRG1, U7 USBLC6-2SC6

Commit message: V2: clear all PCB traces — restart routing from scratch
Removed all 7 remaining routed segments. 57 footprints and 13 copper
zones intact. FB1 (ferrite bead) confirmed clean — L_0402_1005Metric
footprint with 0.38mm pad clearance, DRC violation was from a prior
stale placement now resolved.

Board is now a clean ratsnest ready for routing.

Co-Authored-By: Claude Sonnet 4.6 <noreply@anthropic.com>
Parts:
- FB1: footprint Inductor_SMD:L_01005_0402Metric -> Inductor_SMD:L_0402_1005Metric
- FB2: footprint (none) -> Inductor_SMD:L_0402_1005Metric
Changed lines of the file:
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@@
 	(wire
 		(pts
-			(xy 21.59 81.28) (xy 21.59 84.455)
-		)
-		(stroke
-			(width 0)
-			(type default)
-		)
-	)
-	(wire
-		(pts
 			(xy 124.46 57.15) (xy 125.73 57.15)
 		)
@@
 	(wire
 		(pts
+			(xy 247.65 128.27) (xy 267.97 128.27)
+		)
+		(stroke
+			(width 0)
+			(type default)
+		)
+	)
+	(wire
+		(pts
 			(xy 95.25 30.48) (xy 90.17 30.48)
 		)
@@
 	(wire
 		(pts
-			(xy 247.65 128.27) (xy 262.89 128.27)
-		)
-		(stroke
-			(width 0)
-			(type default)
-		)
-	)
-	(wire
-		(pts
 			(xy 38.1 176.53) (xy 49.53 176.53)
 		)
@@
 	(wire
 		(pts
-			(xy 229.87 152.4) (xy 229.87 148.59)
-		)
-		(stroke
-			(width 0)
-			(type default)
-		)
-	)
-	(wire
-		(pts
 			(xy 87.63 72.39) (xy 88.9 72.39)
 		)
@@
 	(wire
 		(pts
-			(xy 224.79 152.4) (xy 224.79 148.59)
-		)
-		(stroke
-			(width 0)
-			(type default)
-		)
-	)
-	(wire
-		(pts
 			(xy 114.3 22.86) (xy 114.3 24.13)
 		)
@@
 	(wire
 		(pts
-			(xy 29.21 81.28) (xy 29.21 84.455)
-		)
-		(stroke
-			(width 0)
-			(type default)
-		)
-	)
-	(wire
-		(pts
 			(xy 80.01 17.78) (xy 80.01 20.32)
 		)
@@
 	)
 	(label "SPK_P"
-		(at 261.62 128.27 0)
+		(at 267.97 128.27 0)
 		(effects
 			(font
@@
 			)
 		)
-		(property "Footprint" ""
+		(property "Footprint" "Inductor_SMD:L_0402_1005Metric"
 			(at 251.46 132.588 90)
 			(hide yes)
@@
 	(symbol
 		(lib_id "power:GND")
-		(at 224.79 152.4 0)
+		(at 224.79 148.59 0)
 		(unit 1)
 		(body_style 1)
@@
 		(fields_autoplaced yes)
 		(property "Reference" "#PWR029"
-			(at 224.79 158.75 0)
+			(at 224.79 154.94 0)
 			(hide yes)
 			(show_name no)
@@
 		)
 		(property "Value" "GND"
-			(at 224.79 157.48 0)
+			(at 224.79 153.67 0)
 			(show_name no)
 			(do_not_autoplace no)
@@
 		)
 		(property "Footprint" ""
-			(at 224.79 152.4 0)
+			(at 224.79 148.59 0)
 			(hide yes)
 			(show_name no)
@@
 		)
 		(property "Datasheet" ""
-			(at 224.79 152.4 0)
+			(at 224.79 148.59 0)
 			(hide yes)
 			(show_name no)
@@
 		)
 		(property "Description" "Power symbol creates a global label with name \"GND\" , ground"
-			(at 224.79 152.4 0)
+			(at 224.79 148.59 0)
 			(hide yes)
 			(show_name no)
@@
 	(symbol
 		(lib_id "power:GND")
-		(at 29.21 84.455 0)
+		(at 29.21 81.28 0)
 		(unit 1)
 		(body_style 1)
@@
 		(fields_autoplaced yes)
 		(property "Reference" "#PWR02"
-			(at 29.21 90.805 0)
+			(at 29.21 87.63 0)
 			(hide yes)
 			(show_name no)
@@
 		)
 		(property "Value" "GND"
-			(at 29.21 89.535 0)
+			(at 29.21 86.36 0)
 			(show_name no)
 			(do_not_autoplace no)
@@
 		)
 		(property "Footprint" ""
-			(at 29.21 84.455 0)
+			(at 29.21 81.28 0)
 			(hide yes)
 			(show_name no)
@@
 		)
 		(property "Datasheet" ""
-			(at 29.21 84.455 0)
+			(at 29.21 81.28 0)
 			(hide yes)
 			(show_name no)
@@
 		)
 		(property "Description" "Power symbol creates a global label with name \"GND\" , ground"
-			(at 29.21 84.455 0)
+			(at 29.21 81.28 0)
 			(hide yes)
 			(show_name no)
@@
 	(symbol
 		(lib_id "power:GND")
-		(at 229.87 152.4 0)
+		(at 229.87 148.59 0)
 		(unit 1)
 		(body_style 1)
@@
 		(fields_autoplaced yes)
 		(property "Reference" "#PWR030"
-			(at 229.87 158.75 0)
+			(at 229.87 154.94 0)
 			(hide yes)
 			(show_name no)
@@
 		)
 		(property "Value" "GND"
-			(at 229.87 157.48 0)
+			(at 229.87 153.67 0)
 			(show_name no)
 			(do_not_autoplace no)
@@
 		)
 		(property "Footprint" ""
-			(at 229.87 152.4 0)
+			(at 229.87 148.59 0)
 			(hide yes)
 			(show_name no)
@@
 		)
 		(property "Datasheet" ""
-			(at 229.87 152.4 0)
+			(at 229.87 148.59 0)
 			(hide yes)
 			(show_name no)
@@
 		)
 		(property "Description" "Power symbol creates a global label with name \"GND\" , ground"
-			(at 229.87 152.4 0)
+			(at 229.87 148.59 0)
 			(hide yes)
 			(show_name no)
@@
 	(symbol
 		(lib_id "power:GND")
-		(at 21.59 84.455 0)
+		(at 21.59 81.28 0)
 		(unit 1)
 		(body_style 1)
@@
 		(fields_autoplaced yes)
 		(property "Reference" "#PWR01"
-			(at 21.59 90.805 0)
+			(at 21.59 87.63 0)
 			(hide yes)
 			(show_name no)
@@
 		)
 		(property "Value" "GND"
-			(at 21.59 89.535 0)
+			(at 21.59 86.36 0)
 			(show_name no)
 			(do_not_autoplace no)
@@
 		)
 		(property "Footprint" ""
-			(at 21.59 84.455 0)
+			(at 21.59 81.28 0)
 			(hide yes)
 			(show_name no)
@@
 		)
 		(property "Datasheet" ""
-			(at 21.59 84.455 0)
+			(at 21.59 81.28 0)
 			(hide yes)
 			(show_name no)
@@
 		)
 		(property "Description" "Power symbol creates a global label with name \"GND\" , ground"
-			(at 21.59 84.455 0)
+			(at 21.59 81.28 0)
 			(hide yes)
 			(show_name no)
@@
 			)
 		)
-		(property "Footprint" "Inductor_SMD:L_01005_0402Metric"
+		(property "Footprint" "Inductor_SMD:L_0402_1005Metric"
 			(at 243.84 130.048 90)
 			(hide yes)
